File: STM32.kicad_sch (KiCad schematic)
At the start: 33 parts, among them J1 Conn_01x04_Pin, J2 Conn_01x04_Pin, J3 USB_B_Micro, J4 Conn_01x04_Pin, SW1 SW_SPDT, U1 AMS1117-3.3, U2 STM32F411RETx, Y1 8Mhz

Commit message: .
Parts:
- removed C12: 10n, Capacitor_SMD:C_0402_1005Metric, symbol Device:C
- removed C13, C14: 1u, Capacitor_SMD:C_0402_1005Metric, symbol Device:C
- removed FB1: 120R, Inductor_SMD:L_0603_1608Metric, symbol Device:FerriteBead
- added R5: 1k5, Resistor_SMD:R_0402_1005Metric, symbol Device:R
Connections:
- net +3.3VA is gone; now on net +3.3V: U2.13 (VDDA)
- net +3.3V: no longer C3.1, SW1.3 (C), U2.1 (VBAT)
- net GND: now also R4.1, SW1.3 (C), R5.1; no longer SW1.1 (A)
- net NRST: now also SW1.2 (B)
- net SWCLK: now also R5.2
- net VBUS: now also C3.1, U2.1 (VBAT)
- removed net SW_BOOT0: R4.1, SW1.2 (B)
Other:
- note removed: "VDDA Filtering"
- moved on the sheet: C10, C11, C15, C3, C4, C6, C7, C9
